File: testbench/hardware/testbench-hardware.kicad_sch (KiCad schematic)
At the start: 39 parts, among them J1 ZIF DIP-16 Socket, Q1 ZTX458, SW1 Action, SW2 Mode Select, SW3 Enable Power

Commit message: [testbench] pcb layout
Parts:
- D1, D10, D11, D12, D13, D2, D3, D4, D5, D6, D7, D8, D9: footprint (none) -> LED_THT:LED_D3.0mm
- J1: footprint (none) -> Package_DIP:DIP-16_W7.62mm_Socket
- Q1: footprint (none) -> Package_TO_SOT_THT:TO-92_Inline_Wide; symbol Device:Q_NPN_CBE -> Device:Q_NPN_EBC
- R1, R10, R11, R12, R13, R14, R15, R16, R17, R18, R19, R2, R20, R3, R4, R5, R6, R7, R8, R9: footprint (none) -> commons-passives_THT:Passive_THT_resistor_W2.54mm_L12.70mm
- SW1: footprint (none) -> Button_Switch_THT:SW_PUSH-12mm
- SW2, SW3: footprint (none) -> commons-interconnect_THT:g-switch_22f12-gxxx
Connections:
- net +5V: now also Q1.3 (C); no longer Q1.1 (C)
- net Vzif: now also Q1.1 (E); no longer Q1.3 (E)

Commit message: [testbench] start wiring
Connections:
- net B0: now also A1.12 (D9), R16.1; no longer A1.15 (D12), R18.1
- net B1: now also A1.11 (D8), R15.1; no longer A1.26 (A7), R19.1
- net PASTEL: now also R10.1; no longer R12.1
- net R0: now also A1.26 (A7), R20.1; no longer A1.11 (D8), R14.1
- net R1: now also A1.15 (D12), R19.1; no longer A1.12 (D9), R15.1
- net ROUGE: now also R13.1; no longer R9.1
- net V0: now also A1.14 (D11), R18.1; no longer A1.13 (D10), R16.1
- net V1: now also A1.13 (D10); no longer A1.14 (D11)
- net VERT: now also R12.1; no longer R10.1
- net ~{NOIR_INCR}: now also R14.1; no longer R20.1
- net ~{SUPPLT}: now also R9.1; no longer R13.1
- net at A1.18 (AREF): no longer R1.2
- net at A1.19 (A0): now also R1.2
Changed lines of the file:
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@@
   (no_connect (at 115.57 92.71))
   (no_connect (at 133.35 49.53))
-  (no_connect (at 146.05 74.93))
+  (no_connect (at 146.05 69.85))
   (no_connect (at 146.05 80.01))
   (no_connect (at 63.5 176.53))
@@
     (stroke (width 0) (type default))
   )
-  (wire (pts (xy 143.51 69.85) (xy 148.59 69.85))
-    (stroke (width 0) (type default))
-  )
   (wire (pts (xy 40.64 62.23) (xy 48.26 62.23))
     (stroke (width 0) (type default))
@@
     (stroke (width 0) (type default))
   )
+  (wire (pts (xy 148.59 74.93) (xy 143.51 74.93))
+    (stroke (width 0) (type default))
+  )
   (wire (pts (xy 45.72 74.93) (xy 48.26 74.93))
     (stroke (width 0) (type default))
@@
     (stroke (width 0) (type default))
   )
-  (wire (pts (xy 143.51 74.93) (xy 146.05 74.93))
+  (wire (pts (xy 143.51 69.85) (xy 146.05 69.85))
     (stroke (width 0) (type default))
   )
@@
     (stroke (width 0) (type default))
   )
+  (wire (pts (xy 148.59 21.59) (xy 148.59 74.93))
+    (stroke (width 0) (type default))
+  )
   (wire (pts (xy 104.14 133.35) (xy 109.22 133.35))
     (stroke (width 0) (type default))
@@
     (stroke (width 0) (type default))
   )
-  (wire (pts (xy 148.59 21.59) (xy 148.59 69.85))
-    (stroke (width 0) (type default))
-  )
   (bus (pts (xy 125.73 207.01) (xy 125.73 204.47))
     (stroke (width 0) (type default))
@@
     (effects (font (size 1.27 1.27)) (justify right bottom))
   )
-  (label "B1" (at 123.19 238.76 0) (fields_autoplaced)
-    (effects (font (size 1.27 1.27)) (justify left bottom))
-  )
-  (label "V0" (at 105.41 85.09 0) (fields_autoplaced)
+  (label "B1" (at 123.19 228.6 0) (fields_autoplaced)
+    (effects (font (size 1.27 1.27)) (justify left bottom))
+  )
+  (label "V0" (at 105.41 87.63 0) (fields_autoplaced)
     (effects (font (size 1.27 1.27)) (justify left bottom))
   )
@@
     (effects (font (size 1.27 1.27)) (justify right bottom))
   )
-  (label "ROUGE" (at 128.27 201.93 0) (fields_autoplaced)
-    (effects (font (size 1.27 1.27)) (justify left bottom))
-  )
-  (label "VERT" (at 128.27 204.47 0) (fields_autoplaced)
+  (label "ROUGE" (at 128.27 212.09 0) (fields_autoplaced)
+    (effects (font (size 1.27 1.27)) (justify left bottom))
+  )
+  (label "VERT" (at 128.27 209.55 0) (fields_autoplaced)
     (effects (font (size 1.27 1.27)) (justify left bottom))
   )
@@
     (effects (font (size 1.27 1.27)) (justify left bottom))
   )
-  (label "R0" (at 105.41 80.01 0) (fields_autoplaced)
-    (effects (font (size 1.27 1.27)) (justify left bottom))
-  )
-  (label "B0" (at 123.19 236.22 0) (fields_autoplaced)
+  (label "R0" (at 156.21 92.71 180) (fields_autoplaced)
+    (effects (font (size 1.27 1.27)) (justify right bottom))
+  )
+  (label "B0" (at 123.19 231.14 0) (fields_autoplaced)
     (effects (font (size 1.27 1.27)) (justify left bottom))
   )
@@
     (effects (font (size 1.27 1.27)) (justify right bottom))
   )
-  (label "V0" (at 123.19 231.14 0) (fields_autoplaced)
+  (label "V0" (at 123.19 236.22 0) (fields_autoplaced)
     (effects (font (size 1.27 1.27)) (justify left bottom))
   )
@@
     (effects (font (size 1.27 1.27)) (justify left bottom))
   )
-  (label "~{NOIR_INCR}" (at 123.19 241.3 0) (fields_autoplaced)
-    (effects (font (size 1.27 1.27)) (justify left bottom))
-  )
-  (label "R1" (at 123.19 228.6 0) (fields_autoplaced)
+  (label "~{NOIR_INCR}" (at 123.19 226.06 0) (fields_autoplaced)
+    (effects (font (size 1.27 1.27)) (justify left bottom))
+  )
+  (label "R1" (at 123.19 238.76 0) (fields_autoplaced)
     (effects (font (size 1.27 1.27)) (justify left bottom))
   )
@@
     (effects (font (size 1.27 1.27)) (justify left bottom))
   )
-  (label "B1" (at 156.21 92.71 180) (fields_autoplaced)
-    (effects (font (size 1.27 1.27)) (justify right bottom))
-  )
-  (label "R0" (at 123.19 226.06 0) (fields_autoplaced)
-    (effects (font (size 1.27 1.27)) (justify left bottom))
-  )
-  (label "PASTEL" (at 128.27 209.55 0) (fields_autoplaced)
+  (label "B1" (at 105.41 80.01 0) (fields_autoplaced)
+    (effects (font (size 1.27 1.27)) (justify left bottom))
+  )
+  (label "R0" (at 123.19 241.3 0) (fields_autoplaced)
+    (effects (font (size 1.27 1.27)) (justify left bottom))
+  )
+  (label "PASTEL" (at 128.27 204.47 0) (fields_autoplaced)
     (effects (font (size 1.27 1.27)) (justify left bottom))
   )
@@
     (effects (font (size 1.27 1.27)) (justify left bottom))
   )
-  (label "~{SUPPLT}" (at 128.27 212.09 0) (fields_autoplaced)
+  (label "~{SUPPLT}" (at 128.27 201.93 0) (fields_autoplaced)
     (effects (font (size 1.27 1.27)) (justify left bottom))
   )
@@
     (effects (font (size 1.27 1.27)) (justify left bottom))
   )
-  (label "V1" (at 105.41 87.63 0) (fields_autoplaced)
-    (effects (font (size 1.27 1.27)) (justify left bottom))
-  )
-  (label "R1" (at 105.41 82.55 0) (fields_autoplaced)
+  (label "V1" (at 105.41 85.09 0) (fields_autoplaced)
+    (effects (font (size 1.27 1.27)) (justify left bottom))
+  )
+  (label "R1" (at 105.41 90.17 0) (fields_autoplaced)
     (effects (font (size 1.27 1.27)) (justify left bottom))
   )
@@
     (effects (font (size 1.27 1.27)) (justify right bottom))
   )
-  (label "B0" (at 105.41 90.17 0) (fields_autoplaced)
-    (effects (font (size 1.27 1.27)) (justify left bottom))
-  )
+  (label "B0" (at 105.41 82.55 0) (fields_autoplaced)
+    (effects (font (size 1.27 1.27)) (justify left bottom))
+  )

Commit message: [testbench] mounting holes
Parts:
- added H1, H2: M2.5, MountingHole:MountingHole_2.7mm_M2.5, symbol Mechanical:MountingHole
Changed lines of the file:
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@@
+    )
+  )
+  (symbol (lib_id "Mechanical:MountingHole") (at 59.69 241.3 0) (unit 1)
+    (in_bom yes) (on_board yes) (dnp no)
+    (property "Reference" "H2" (at 59.69 236.22 0)
+      (effects (font (size 1.27 1.27)))
+    )
+    (property "Value" "M2.5" (at 59.69 238.125 0)
+      (effects (font (size 1.27 1.27)))
+    )
+    (property "Footprint" "MountingHole:MountingHole_2.7mm_M2.5" (at 59.69 241.3 0)
+      (effects (font (size 1.27 1.27)) hide)
+    )
+    (property "Datasheet" "~" (at 59.69 241.3 0)
+      (effects (font (size 1.27 1.27)) hide)
+    )
+    (instances
+      (project "testbench-hardware"
+        (path "/b9af5566-2060-4517-99e4-3893ebe5c065"
+          (reference "H2") (unit 1)
+        )
+      )
     )
   )
@@
         )
       )
+    )
+  )
+  (symbol (lib_id "Mechanical:MountingHole") (at 52.07 241.3 0) (unit 1)
+    (in_bom yes) (on_board yes) (dnp no)
+    (property "Reference" "H1" (at 52.07 236.22 0)
+      (effects (font (size 1.27 1.27)))
+    )
+    (property "Value" "M2.5" (at 52.07 238.125 0)
+      (effects (font (size 1.27 1.27)))
+    )
+    (property "Footprint" "MountingHole:MountingHole_2.7mm_M2.5" (at 52.07 241.3 0)
+      (effects (font (size 1.27 1.27)) hide)
+    )
+    (property "Datasheet" "~" (at 52.07 241.3 0)
+      (effects (font (size 1.27 1.27)) hide)
+    )
+    (instances
+      (project "testbench-hardware"
+        (path "/b9af5566-2060-4517-99e4-3893ebe5c065"
+          (reference "H1") (unit 1)
+        )
+      )

Commit message: [testbench] uses DPDT switches as SPDT switches for nicer routing
Parts:
- SW2, SW3: footprint commons-interconnect_THT:g-switch_22f12-gxxx -> commons-interconnect_THT:g-switch_22f12-gxxx--SPDT
Changed lines of the file:
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@@
       (effects (font (size 1.27 1.27)))
     )
-    (property "Footprint" "commons-interconnect_THT:g-switch_22f12-gxxx" (at 83.82 138.43 0)
+    (property "Footprint" "commons-interconnect_THT:g-switch_22f12-gxxx--SPDT" (at 83.82 138.43 0)
       (effects (font (size 1.27 1.27)) hide)
     )
@@
       (effects (font (size 1.27 1.27)))
     )
-    (property "Footprint" "commons-interconnect_THT:g-switch_22f12-gxxx" (at 71.12 163.83 0)
+    (property "Footprint" "commons-interconnect_THT:g-switch_22f12-gxxx--SPDT" (at 71.12 163.83 0)
       (effects (font (size 1.27 1.27)) hide)
     )

Commit message: Fixes #2 : [bug][testbench][hardware] A6 and A7 cannot be used as digital input
Connections:
- net R0: now also A1.20 (A1); no longer A1.26 (A7)
- net at A1.25 (A6): no longer R3.2
- net POWER_ENABLE_SWITCH: now reaches A1.23 (A4), R7.2
- net ACTION_BUTTON: now reaches A1.21 (A2)
- net ACTION_BUTTON: now also R3.2
- net MODE_SWITCH: now reaches A1.24 (A5), R5.2
Other:
- moved on the sheet: R3, R4, R5, R6, R7, R8, SW1, SW2, SW3

Commit message: Fixes #3 : [bug][testbench] remove R3, R5 and R7
Parts:
- removed R3, R5, R7: 10K, commons-passives_THT:Passive_THT_resistor_W2.54mm_L12.70mm, symbol Device:R_Small_US
Connections:
- net ACTION_BUTTON: now also R4.2, SW1.2
- net MODE_SWITCH: now also R6.2, SW2.2 (B)
- net POWER_ENABLE_SWITCH: now also R8.2, SW3.2 (B)
Changed lines of the file:
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@@
-    (stroke (width 0) (type default))
-  )
-  (wire (pts (xy 114.3 116.84) (xy 121.92 116.84))
     (stroke (width 0) (type default))
   )
@@
     (stroke (width 0) (type default))
   )
-  (wire (pts (xy 127 134.62) (xy 180.34 134.62))
+  (wire (pts (xy 114.3 134.62) (xy 180.34 134.62))
     (stroke (width 0) (type default))
   )
@@
     (stroke (width 0) (type default))
   )
-  (wire (pts (xy 127 152.4) (xy 185.42 152.4))
+  (wire (pts (xy 114.3 152.4) (xy 185.42 152.4))
     (stroke (width 0) (type default))
   )
@@
     (stroke (width 0) (type default))
   )
-  (wire (pts (xy 114.3 152.4) (xy 121.92 152.4))
-    (stroke (width 0) (type default))
-  )
   (wire (pts (xy 165.1 201.93) (xy 173.99 201.93))
     (stroke (width 0) (type default))
@@
     (stroke (width 0) (type default))
   )
-  (wire (pts (xy 114.3 134.62) (xy 121.92 134.62))
-    (stroke (width 0) (type default))
-  )
   (bus (pts (xy 38.1 59.69) (xy 38.1 62.23))
     (stroke (width 0) (type default))
@@
     (stroke (width 0) (type default))
   )
-  (wire (pts (xy 127 116.84) (xy 175.26 116.84))
+  (wire (pts (xy 114.3 116.84) (xy 175.26 116.84))
     (stroke (width 0) (type default))
   )
@@
         (path "/b9af5566-2060-4517-99e4-3893ebe5c065"
           (reference "R11") (unit 1)
-        )
-      )
-    )
-  )
-  (symbol (lib_id "Device:R_Small_US") (at 124.46 152.4 90) (unit 1)
-    (in_bom yes) (on_board yes) (dnp no)
-    (property "Reference" "R3" (at 121.92 151.13 90)
-      (effects (font (size 1.27 1.27)) (justify left))
-    )
-    (property "Value" "10K" (at 127 151.13 90)
-      (effects (font (size 1.27 1.27)) (justify right))
-    )
-    (property "Footprint" "commons-passives_THT:Passive_THT_resistor_W2.54mm_L12.70mm" (at 124.46 152.4 0)
-      (effects (font (size 1.27 1.27)) hide)
-    )
-    (property "Datasheet" "~" (at 124.46 152.4 0)
-      (effects (font (size 1.27 1.27)) hide)
-    )
-    (pin "2")
-    (pin "1")
-    (instances
-      (project "testbench-hardware"
-        (path "/b9af5566-2060-4517-99e4-3893ebe5c065"
-          (reference "R3") (unit 1)
         )
       )
@@
         (path "/b9af5566-2060-4517-99e4-3893ebe5c065"
           (reference "D6") (unit 1)
-        )
-      )
-    )
-  )
-  (symbol (lib_id "Device:R_Small_US") (at 124.46 134.62 90) (unit 1)
-    (in_bom yes) (on_board yes) (dnp no)
-    (property "Reference" "R7" (at 121.92 133.35 90)
-      (effects (font (size 1.27 1.27)) (justify left))
-    )
-    (property "Value" "10K" (at 127 133.35 90)
-      (effects (font (size 1.27 1.27)) (justify right))
-    )
-    (property "Footprint" "commons-passives_THT:Passive_THT_resistor_W2.54mm_L12.70mm" (at 124.46 134.62 0)
-      (effects (font (size 1.27 1.27)) hide)
-    )
-    (property "Datasheet" "~" (at 124.46 134.62 0)
-      (effects (font (size 1.27 1.27)) hide)
-    )
-    (pin "2")
-    (pin "1")
-    (instances
-      (project "testbench-hardware"
-        (path "/b9af5566-2060-4517-99e4-3893ebe5c065"
-          (reference "R7") (unit 1)
         )
       )
@@
         )
       )
-    )
-  )
-  (symbol (lib_id "Device:R_Small_US") (at 124.46 116.84 90) (unit 1)
-    (in_bom yes) (on_board yes) (dnp no)
-    (property "Reference" "R5" (at 121.92 115.57 90)
-      (effects (font (size 1.27 1.27)) (justify left))
-    )
-    (property "Value" "10K" (at 127 115.57 90)
-      (effects (font (size 1.27 1.27)) (justify right))
-    )
-    (property "Footprint" "commons-passives_THT:Passive_THT_resistor_W2.54mm_L12.70mm" (at 124.46 116.84 0)
-      (effects (font (size 1.27 1.27)) hide)
-    )
-    (property "Datasheet" "~" (at 124.46 116.84 0)
-      (effects (font (size 1.27 1.27)) hide)
-    )
-    (pin "2")
-    (pin "1")
-    (instances
-      (project "testbench-hardware"
-        (path "/b9af5566-2060-4517-99e4-3893ebe5c065"
-          (reference "R5") (unit 1)
-        )
-      )

Commit message: Resolves #5 : [testbench][hardware] Change Q1 to a Darlington
Parts:
- Q1: value ZTX458 -> KSP13TA; symbol Device:Q_NPN_EBC -> Device:Q_NPN_Darlington_EBC
Changed lines of the file:
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@@
     )
   )
-  (symbol (lib_id "Device:Q_NPN_EBC") (at 76.2 30.48 270) (unit 1)
+  (symbol (lib_id "Device:Q_NPN_Darlington_EBC") (at 76.2 30.48 270) (unit 1)
     (in_bom yes) (on_board yes) (dnp no)
     (property "Reference" "Q1" (at 80.01 29.21 90)
       (effects (font (size 1.27 1.27)) (justify left))
     )
-    (property "Value" "ZTX458" (at 80.01 31.75 90)
+    (property "Value" "KSP13TA" (at 80.01 31.75 90)
       (effects (font (size 1.27 1.27)) (justify left))
     )
